Commit message: ✨ feat: 使scara固定在地面

File: src/scara_robot_description/urdf/gazebo.xacro (robot description, xacro)
@@ -1,4 +1,10 @@
 <robot name="base" xmlns:xacro="http://wiki.ros.org/xacro">
     <xacro:include filename="scara.xacro" />
+    <link name="world"/>
+    <joint name="base_2_world" type="fixed">
+        <parent link="world"/>
+        <child link="base_link"/>
+        <origin xyz="0.0 0.0 ${base_link_z/2}"/>
+    </joint>
     <gazebo reference="base_link">
         <material>Gazebo/Red</material>

Commit message: ✨ feat: 添加transmission元素

File: src/scara_robot_description/urdf/gazebo.xacro (robot description, xacro)
@@ -1,9 +1,9 @@
 <robot name="base" xmlns:xacro="http://wiki.ros.org/xacro">
     <xacro:include filename="scara.xacro" />
-    <link name="world"/>
+    <link name="world" />
     <joint name="base_2_world" type="fixed">
-        <parent link="world"/>
-        <child link="base_link"/>
-        <origin xyz="0.0 0.0 ${base_link_z/2}"/>
+        <parent link="world" />
+        <child link="base_link" />
+        <origin xyz="0.0 0.0 ${base_link_z/2}" />
     </joint>
     <gazebo reference="base_link">
@@ -28,3 +28,68 @@
         <material>Gazebo/Blue</material>
     </gazebo>
+    <gazebo>
+        <plugin name="gazebo_ros_control" filename="libgazebo_ros_control.so">
+            <robotNamespace>/rrbot</robotNamespace>
+        </plugin>
+    </gazebo>
+    <transmission name="tran1">
+        <type>transmission_interface/SimpleTransmission</type>
+        <joint name="link12base">
+            <hardwareInterface>hardware_interface/PositionJointInterface</hardwareInterface>
+        </joint>
+        <actuator name="motor1">
+            <hardwareInterface>hardware_interface/PositionJointInterface</hardwareInterface>
+            <mechanicalReduction>1</mechanicalReduction>
+        </actuator>
+    </transmission>
+    <transmission name="tran2">
+        <type>transmission_interface/SimpleTransmission</type>
+        <joint name="link2_to_link1">
+            <hardwareInterface>hardware_interface/PositionJointInterface</hardwareInterface>
+        </joint>
+        <actuator name="motor2">
+            <hardwareInterface>hardware_interface/PositionJointInterface</hardwareInterface>
+            <mechanicalReduction>1</mechanicalReduction>
+        </actuator>
+    </transmission>
+    <transmission name="tran3">
+        <type>transmission_interface/SimpleTransmission</type>
+        <joint name="link3_to_link2">
+            <hardwareInterface>hardware_interface/PositionJointInterface</hardwareInterface>
+        </joint>
+        <actuator name="motor3">
+            <hardwareInterface>hardware_interface/PositionJointInterface</hardwareInterface>
+            <mechanicalReduction>1</mechanicalReduction>
+        </actuator>
+    </transmission>
+    <transmission name="tran4">
+        <type>transmission_interface/SimpleTransmission</type>
+        <joint name="gripper_base_link_to_link3">
+            <hardwareInterface>hardware_interface/PositionJointInterface</hardwareInterface>
+        </joint>
+        <actuator name="motor4">
+            <hardwareInterface>hardware_interface/PositionJointInterface</hardwareInterface>
+            <mechanicalReduction>1</mechanicalReduction>
+        </actuator>
+    </transmission>
+    <transmission name="tran5">
+        <type>transmission_interface/SimpleTransmission</type>
+        <joint name="left_2_gripper_base">
+            <hardwareInterface>hardware_interface/PositionJointInterface</hardwareInterface>
+        </joint>
+        <actuator name="motor5">
+            <hardwareInterface>hardware_interface/PositionJointInterface</hardwareInterface>
+            <mechanicalReduction>1</mechanicalReduction>
+        </actuator>
+    </transmission>
+    <transmission name="tran6">
+        <type>transmission_interface/SimpleTransmission</type>
+        <joint name="right_2_gripper_base">
+            <hardwareInterface>hardware_interface/PositionJointInterface</hardwareInterface>
+        </joint>
+        <actuator name="motor6">
+            <hardwareInterface>hardware_interface/PositionJointInterface</hardwareInterface>
+            <mechanicalReduction>1</mechanicalReduction>
+        </actuator>
+    </transmission>
 </robot>

Commit message: 📃 docs: joint命名规范

File: src/scara_robot_description/urdf/gazebo.xacro (robot description, xacro)
@@ -2,5 +2,5 @@
     <xacro:include filename="scara.xacro" />
     <link name="world" />
-    <joint name="base_2_world" type="fixed">
+    <joint name="base_to_world" type="fixed">
         <parent link="world" />
         <child link="base_link" />
@@ -35,5 +35,5 @@
     <transmission name="tran1">
         <type>transmission_interface/SimpleTransmission</type>
-        <joint name="link12base">
+        <joint name="link1_to_base">
             <hardwareInterface>hardware_interface/PositionJointInterface</hardwareInterface>
         </joint>
@@ -75,5 +75,5 @@
     <transmission name="tran5">
         <type>transmission_interface/SimpleTransmission</type>
-        <joint name="left_2_gripper_base">
+        <joint name="left_to_gripper_base">
             <hardwareInterface>hardware_interface/PositionJointInterface</hardwareInterface>
         </joint>
@@ -85,5 +85,5 @@
     <transmission name="tran6">
         <type>transmission_interface/SimpleTransmission</type>
-        <joint name="right_2_gripper_base">
+        <joint name="right_to_gripper_base">
             <hardwareInterface>hardware_interface/PositionJointInterface</hardwareInterface>
         </joint>

File: src/scara_robot_description/urdf/scara.xacro (robot description, xacro)
@@ -45,5 +45,5 @@
         <xacro:cylinder_inertial_matrix m="${link1_m}" r="${link1_radius}" h="${link1_length}" />
     </link>
-    <joint name="link12base" type="revolute">
+    <joint name="link1_to_base" type="revolute">
         <parent link="base_link" />
         <child link="link1" />
@@ -175,5 +175,5 @@
             w="${gripper_finger_link_y}" h="${gripper_finger_link_z}" />
     </link>
-    <joint name="left_2_gripper_base" type="prismatic">
+    <joint name="left_to_gripper_base" type="prismatic">
         <parent link="gripper_base_link" />
         <child link="gripper_left" />
@@ -205,5 +205,5 @@
             w="${gripper_finger_link_y}" h="${gripper_finger_link_z}" />
     </link>
-    <joint name="right_2_gripper_base" type="prismatic">
+    <joint name="right_to_gripper_base" type="prismatic">
         <parent link="gripper_base_link" />
         <child link="gripper_right" />

Commit message: 🐞 fix(删除transmission):

File: src/scara_robot_description/urdf/gazebo.xacro (robot description, xacro)
@@ -30,66 +30,6 @@
     <gazebo>
         <plugin name="gazebo_ros_control" filename="libgazebo_ros_control.so">
-            <robotNamespace>/rrbot</robotNamespace>
+            <robotNamespace>/scara_robot</robotNamespace>
         </plugin>
     </gazebo>
-    <transmission name="tran1">
-        <type>transmission_interface/SimpleTransmission</type>
-        <joint name="link1_to_base">
-            <hardwareInterface>hardware_interface/PositionJointInterface</hardwareInterface>
-        </joint>
-        <actuator name="motor1">
-            <hardwareInterface>hardware_interface/PositionJointInterface</hardwareInterface>
-            <mechanicalReduction>1</mechanicalReduction>
-        </actuator>
-    </transmission>
-    <transmission name="tran2">
-        <type>transmission_interface/SimpleTransmission</type>
-        <joint name="link2_to_link1">
-            <hardwareInterface>hardware_interface/PositionJointInterface</hardwareInterface>
-        </joint>
-        <actuator name="motor2">
-            <hardwareInterface>hardware_interface/PositionJointInterface</hardwareInterface>
-            <mechanicalReduction>1</mechanicalReduction>
-        </actuator>
-    </transmission>
-    <transmission name="tran3">
-        <type>transmission_interface/SimpleTransmission</type>
-        <joint name="link3_to_link2">
-            <hardwareInterface>hardware_interface/PositionJointInterface</hardwareInterface>
-        </joint>
-        <actuator name="motor3">
-            <hardwareInterface>hardware_interface/PositionJointInterface</hardwareInterface>
-            <mechanicalReduction>1</mechanicalReduction>
-        </actuator>
-    </transmission>
-    <transmission name="tran4">
-        <type>transmission_interface/SimpleTransmission</type>
-        <joint name="gripper_base_link_to_link3">
-            <hardwareInterface>hardware_interface/PositionJointInterface</hardwareInterface>
-        </joint>
-        <actuator name="motor4">
-            <hardwareInterface>hardware_interface/PositionJointInterface</hardwareInterface>
-            <mechanicalReduction>1</mechanicalReduction>
-        </actuator>
-    </transmission>
-    <transmission name="tran5">
-        <type>transmission_interface/SimpleTransmission</type>
-        <joint name="left_to_gripper_base">
-            <hardwareInterface>hardware_interface/PositionJointInterface</hardwareInterface>
-        </joint>
-        <actuator name="motor5">
-            <hardwareInterface>hardware_interface/PositionJointInterface</hardwareInterface>
-            <mechanicalReduction>1</mechanicalReduction>
-        </actuator>
-    </transmission>
-    <transmission name="tran6">
-        <type>transmission_interface/SimpleTransmission</type>
-        <joint name="right_to_gripper_base">
-            <hardwareInterface>hardware_interface/PositionJointInterface</hardwareInterface>
-        </joint>
-        <actuator name="motor6">
-            <hardwareInterface>hardware_interface/PositionJointInterface</hardwareInterface>
-            <mechanicalReduction>1</mechanicalReduction>
-        </actuator>
-    </transmission>
 </robot>
